File: electronics/kicad/standalonepanel/standalonepanel.kicad_pcb (KiCad board)
At the start: 2 copper layers, 135 x 54 mm, 110 parts, among them J1 LEDPWR, J2 USB_C-PD, J3 Speaker, Q1 AO4435, SW1 SET, SW2 BOOT, SW3 UP, SW4 DOWN, SW5 TST-ICE40, SW6 RESET, U1 SC189ZSKTRT, U10 DS3231, U11 SN74LVC8T245, U12 SN74LVC8T245, U13 SN74LVC8T245, U2 SC189CSKTRT, U3 CH340C, U4 ESP32-WROVER-E, U5 IS64WV25616EFBLL-10TLI, U6 STUSB4500QTR, U7 ICE40-HX4K, U8 MAX98357A, U9 MPU-6050, X1 12MHz

Commit message: v3 of electronics
Parts:
- removed C15, C16, C19, C20, C21: 1uF, Capacitor_SMD:C_0805_2012Metric_Pad1.18x1.45mm_HandSolder
- removed C25: 100nF, Capacitor_SMD:C_0805_2012Metric_Pad1.18x1.45mm_HandSolder
- removed D1, D4, D5, D6: P4SMA27A, Diode_SMD:D_SMA_Handsoldering
- removed D3: BAT760, Diode_SMD:D_SOD-323
- removed LED4: PD, LED_SMD:LED_1206_3216Metric_Pad1.42x1.75mm_HandSolder
- removed Q1: AO4435, Package_SO:SOIC-8_3.9x4.9mm_P1.27mm
- removed R14: 22K, Resistor_SMD:R_1206_3216Metric_Pad1.30x1.75mm_HandSolder
- removed R15: 1K, Resistor_SMD:R_1206_3216Metric_Pad1.30x1.75mm_HandSolder
- removed R16: 1K5, Resistor_SMD:R_1206_3216Metric_Pad1.30x1.75mm_HandSolder
- removed R17: 10K, Resistor_SMD:R_1206_3216Metric_Pad1.30x1.75mm_HandSolder
- removed U8: MAX98357A, Package_DFN_QFN:TQFN-16-1EP_3x3mm_P0.5mm_EP1.6x1.6mm
- removed U9: MPU-6050, 0_project:InvenSense_QFN-24_4x4mm_P0.5mm
- added C46: 100nF, Capacitor_SMD:C_0805_2012Metric_Pad1.18x1.45mm_HandSolder, B.Cu at (130.2, 101.7)
- added C47: 100nF, Capacitor_SMD:C_0805_2012Metric_Pad1.18x1.45mm_HandSolder, B.Cu at (119.4, 103.9)
- added J4: Conn_01x07_Pin, Connector_PinHeader_2.54mm:PinHeader_1x07_P2.54mm_Vertical, F.Cu at (139.5, 125.0)
- added JP1: 3V3, Jumper:SolderJumper-2_P1.3mm_Open_RoundedPad1.0x1.5mm, F.Cu at (80.0, 118.0)
- added JP2: 1V2, Jumper:SolderJumper-2_P1.3mm_Open_RoundedPad1.0x1.5mm, F.Cu at (80.0, 122.9)
- BT1: footprint 0_project:cr2032_smd_clip -> 0_whitemagic:cr2032_smd_clip
- C12, C33, C42, C44, R8, U11, U12, U13: moved to B.Cu
- C14: value 100nF -> 470uF; footprint Capacitor_SMD:C_0805_2012Metric_Pad1.18x1.45mm_HandSolder -> Capacitor_SMD:C_Elec_8x10.2
- C28: value 10uF -> 100nF
- C29: value 100nF -> 10uF
- C32: value 10nF -> 100nF; moved to B.Cu
- C43: value 2.2nF/50V -> 100nF; moved to B.Cu
- G***: footprint 0_project:white_magic -> 0_whitemagic:white_magic
- HUB75E-1, HUB75E-2: footprint 0_project:IDC-Header_2x08_P2.54mm_Horizontal -> 0_whitemagic:IDC-Header_2x08_P2.54mm_Horizontal
- J1: footprint 0_project:JST_VH_1x04_P3.96mm_Horizontal -> 0_whitemagic:JST_VH_1x04_P3.96mm_Horizontal
- J2: footprint 0_project:USB_C_Receptacle_G-Switch_GT-USB-7010ASV -> 0_whitemagic:USB_C_Receptacle_G-Switch_GT-USB-7010ASV
- L1, L2: footprint 0_project:Inductor-040420 -> 0_whitemagic:Inductor-040420
- R10: value 100K -> 390R
- R11: value 1K -> 390R
- R12: value 100R -> 4K7
- R13: value 470R -> 4K7
- R2: value 10K -> 2K2
- R5: value 2K2 -> 10K
- SW1: value SET -> UP; footprint 0_project:SW_Tactile_SKHH_Angled -> 0_whitemagic:SW_Tactile_SKHH_Angled
- SW3: value UP -> SET; footprint 0_project:SW_Tactile_SKHH_Angled -> 0_whitemagic:SW_Tactile_SKHH_Angled
- SW4: footprint 0_project:SW_Tactile_SKHH_Angled -> 0_whitemagic:SW_Tactile_SKHH_Angled
- U1, U2: footprint 0_project:SOT23-5-SC189_SEM -> 0_whitemagic:SOT23-5-SC189_SEM
- U4: footprint 0_project:ESP32-WROVER-E -> 0_whitemagic:ESP32-WROVER-E
- U6: value STUSB4500QTR -> MAX98357A; footprint 0_project:QFN-24-1EP_4x4mm_P0.5mm_EP2.7x2.7mm -> Package_DFN_QFN:TQFN-16-1EP_3x3mm_P0.5mm_EP1.6x1.6mm
- X1: footprint 0_project:Oscillator_SMD_EuroQuartz_XO91-4Pin_7.0x5.0mm_HandSoldering -> 0_whitemagic:Oscillator_SMD_EuroQuartz_XO91-4Pin_7.0x5.0mm_HandSoldering
- moved R5 109.3 mm to (54.5, 112.0)
- moved C32 66.5 mm to (108.5, 94.5), turned to 90 degrees
- moved R2 58.9 mm to (165.4, 116.8), turned to 0 degrees
- moved C33 58.1 mm to (111.3, 103.7), turned to 180 degrees
- moved R6 57.6 mm to (54.5, 122.5), turned to 90 degrees
- moved R7 53.4 mm to (54.6, 130.2), turned to 90 degrees
- moved U13 52.6 mm to (113.8, 98.2), turned to -90 degrees
- moved SW4 50.9 mm to (48.8, 134.4), turned to 90 degrees
- moved R9 48.5 mm to (86.8, 120.8)
- moved SW3 43.7 mm to (48.8, 124.4), turned to 90 degrees
- moved C42 43.1 mm to (128.3, 104.7), turned to 180 degrees
- moved G*** 41.3 mm to (89.5, 138.8)
- moved SW1 40.5 mm to (48.8, 114.4), turned to 90 degrees
- moved LED3 38.6 mm to (86.0, 116.2), turned to 90 degrees
- moved C12 37.5 mm to (60.1, 130.5)
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Connections:
- C14 pad 1: VPANEL -> VBUS
- C14 pad 2: Net-(C14-Pad2) -> GND
- C32 pad 1: GND -> VBUS
- C32 pad 2: +3V3 -> GND
- C4 pad 1: +3V3 -> Net-(JP1-A)
- C42 pad 2: Net-(U9-REGOUT) -> +3V3
- C43 pad 1: GND -> VBUS
- C43 pad 2: Net-(U9-CPOUT) -> GND
- C6 pad 1: +1V2 -> Net-(JP2-A)
- J1 pad 1: VPANEL -> VBUS
- J1 pad 2: VPANEL -> VBUS
- J2 pad A5: Net-(D5-K) -> Net-(J2-CC1)
- J2 pad B5: Net-(D6-K) -> Net-(J2-CC2)
- L1 pad 2: +3V3 -> Net-(JP1-A)
- L2 pad 2: +1V2 -> Net-(JP2-A)
- R1 pad 2: +3V3 -> Net-(JP1-A)
- R10 pad 1: VBUS -> Net-(R10-Pad1)
- R10 pad 2: Net-(Q1-G1) -> Net-(J2-CC2)
- R11 pad 1: VPANEL -> Net-(R11-Pad1)
- R11 pad 2: Net-(U6-DISCH) -> Net-(J2-CC1)
- R12 pad 1: Net-(C14-Pad2) -> GND
- R12 pad 2: Net-(Q1-G1) -> Net-(R11-Pad1)
- R13 pad 1: VBUS -> GND
- R13 pad 2: Net-(D3-K) -> Net-(R10-Pad1)
- R2 pad 1: +3V3 -> Net-(U4-32K_XN/GPIO33/ADC1_CH5)
- R2 pad 2: Net-(U4-32K_XP/GPIO32/ADC1_CH4) -> Net-(LED2-A)
- R5 pad 1: Net-(U4-32K_XN/GPIO33/ADC1_CH5) -> +3V3
- R5 pad 2: Net-(LED2-A) -> Net-(U4-32K_XP/GPIO32/ADC1_CH4)
- U1 pad 4: +3V3 -> Net-(JP1-A)
- U11 pad 1: +3V3 -> VBUS
- U11 pad 23: VBUS -> +3V3
- U11 pad 24: VBUS -> +3V3
- U12 pad 1: +3V3 -> VBUS
- U12 pad 23: VBUS -> +3V3
- U12 pad 24: VBUS -> +3V3
- U13 pad 1: +3V3 -> VBUS
- U13 pad 10: DSP-LAT-5V -> DSP-E-5V
- U13 pad 14: DSP-LAT -> DSP-E
- U13 pad 15: DSP-OE -> DSP-A
- U13 pad 16: DSP-CLK -> DSP-B
- U13 pad 17: DSP-E -> DSP-C
- U13 pad 19: DSP-C -> DSP-CLK
- U13 pad 20: DSP-B -> DSP-LAT
- U13 pad 21: DSP-A -> DSP-OE
- U13 pad 23: VBUS -> +3V3
- U13 pad 24: VBUS -> +3V3
- U13 pad 3: DSP-A-5V -> DSP-OE-5V
- U13 pad 4: DSP-B-5V -> DSP-LAT-5V
- U13 pad 5: DSP-C-5V -> DSP-CLK-5V
- U13 pad 7: DSP-E-5V -> DSP-C-5V
- U13 pad 8: DSP-CLK-5V -> DSP-B-5V
- U13 pad 9: DSP-OE-5V -> DSP-A-5V
- U2 pad 4: +1V2 -> Net-(JP2-A)
- U6 pad 1: Net-(D5-K) -> Net-(U6-DIN)
- U6 pad 10: GND -> Net-(J3-Pin_2)
- U6 pad 11: unconnected-(U6-ATTACH-Pad11) -> GND
- U6 pad 12: GND -> unconnected-(U6-NC-Pad12)
- U6 pad 13: GND -> unconnected-(U6-NC-Pad13)
- U6 pad 14: unconnected-(U6-POWER_OK3-Pad14) -> Net-(U6-LRCLK)
- U6 pad 15: unconnected-(U6-GPIO-Pad15) -> GND
- U6 pad 16: Net-(U6-VBUS_EN_SNK) -> Net-(U6-BCLK)
- U6 pad 17: unconnected-(U6-A_B_SIDE-Pad17) -> (no net)
- U6 pad 2: Net-(D5-K) -> GND
- U6 pad 3: unconnected-(U6-NC-Pad3) -> GND
- U6 pad 4: Net-(D6-K) -> Net-(U6-~{SD_MODE})
- U6 pad 5: Net-(D6-K) -> unconnected-(U6-NC-Pad5)
- U6 pad 6: Net-(U6-RESET) -> unconnected-(U6-NC-Pad6)
- U6 pad 7: I2C-CLK -> +3V3
- U6 pad 8: I2C-SDA -> +3V3
- U6 pad 9: Net-(U6-DISCH) -> Net-(J3-Pin_1)
- U7 pad 1: unconnected-(U7-IOL_2A-Pad1) -> Net-(U6-~{SD_MODE})
- U7 pad 124: DSP-E -> DSP1-B2
- U7 pad 125: DSP1-B2 -> DSP-E
- U7 pad 144: Net-(LED3-A) -> unconnected-(U7-IOT_222-Pad144)
- U7 pad 15: Net-(U7-IOL_10A) -> unconnected-(U7-IOL_10A-Pad15)
- U7 pad 16: Net-(U7-IOL_10B) -> unconnected-(U7-IOL_10B-Pad16)
- U7 pad 17: Net-(U7-IOL_12A) -> unconnected-(U7-IOL_12A-Pad17)
- U7 pad 18: Net-(U7-IOL_12B) -> unconnected-(U7-IOL_12B-Pad18)
- U7 pad 2: unconnected-(U7-IOL_2B-Pad2) -> Net-(U6-DIN)
- U7 pad 3: unconnected-(U7-IOL_3A-Pad3) -> Net-(U6-BCLK)
- U7 pad 4: unconnected-(U7-IOL_3B-Pad4) -> Net-(U6-LRCLK)
- U7 pad 7: unconnected-(U7-IOL_4A-Pad7) -> Net-(LED3-A)
Routing:
- net I2C-SDA: track 180.7 -> 50.7 mm, vias 6 -> 2
- net DSP-OE-5V: track 0.00 -> 129.3 mm, vias 0 -> 2
- net I2C-CLK: track 182.5 -> 54.0 mm, vias 6 -> 2
- net DSP-CLK-5V: track 0.00 -> 125.6 mm, vias 0 -> 2
- net DSP-C-5V: track 0.00 -> 122.8 mm, vias 0 -> 2
- net DSP-LAT-5V: track 0.00 -> 121.1 mm, vias 0 -> 2
- net DSP-A-5V: track 0.00 -> 119.4 mm, vias 0 -> 2
- net DSP-D-5V: track 0.00 -> 118.2 mm, vias 0 -> 2
- net DSP-B-5V: track 0.00 -> 115.0 mm, vias 0 -> 2
- net DSP-E-5V: track 0.00 -> 111.2 mm, vias 0 -> 2
- net VPANEL: track 99.7 -> 0.00 mm, vias 2 -> 0
- net VBUS: track 114.7 -> 213.0 mm, vias 3 -> 6
- net DSP-A: track 108.5 -> 19.8 mm
- net DSP-E: track 105.8 -> 18.5 mm
- net DSP-B: track 103.7 -> 19.3 mm
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Other:
- board text added: "+5V"
- board text added: "3v3"
- board text added: "CLK"
- board text added: "SCK"
- board text added: "SDA"
- board text added: "SDI"
- board text added: "SDO"
- board text added: "Standalonepanel v3 EvO Dec 2024"
- board text added: "battery"
- board text removed: "+++"
- board text removed: "Standalonepanel v2 EvO Sep 2024"
